Commit message: Add mod to get a basic simulation with only shoulder

File: robots_description/models/aeroarms/arm.transmission.xacro (robot description, xacro)
@@ -16,11 +16,11 @@
   <!-- Left arm -->
   <qside_x_transmission side="1" x="1"/>
-  <qside_x_transmission side="1" x="2"/>
-  <qside_x_transmission side="1" x="3"/>
-  <qside_x_transmission side="1" x="4"/>
+  <!-- <qside_x_transmission side="1" x="2"/> -->
+  <!-- <qside_x_transmission side="1" x="3"/>
+  <qside_x_transmission side="1" x="4"/> -->
   <!-- Right arm -->
-  <qside_x_transmission side="2" x="1"/>
+  <!-- <qside_x_transmission side="2" x="1"/>
   <qside_x_transmission side="2" x="2"/>
   <qside_x_transmission side="2" x="3"/>
-  <qside_x_transmission side="2" x="4"/>
+  <qside_x_transmission side="2" x="4"/> -->
 </robot>

File: robots_description/models/aeroarms/geometry.xacro (robot description, xacro)
@@ -115,13 +115,11 @@
     <parent link="base_link"/>
     <child link="left_shoulder"/>
-    <axis xyz="0 0 1"/>
+    <axis xyz="0 1 0"/>
     <dynamics damping="0.7" friction="0.4"/>
     <limit effort="5000.0" lower="${-0.5*pi}" upper="${0.5*pi}" velocity="1"/>
   </joint>
-  <link name="left_upperarm">
+  <!-- <link name="left_upperarm">
     <inertial>
       <origin xyz="-10.426e-3 -26.142e-3 -82.655e-3"/>
-      <!--mass value="0.245"/>
-      <inertia ixx="4.61e-04" ixy="7.12e-07" ixz="1.96e-05" iyy="4.81e-04" iyz="7.44e-07" izz="9.37e-05"/-->
       <mass value="0.1"/>
       <inertia ixx="8.5833e-04" ixy="0" ixz="0" iyy="8.5833e-04" iyz="0" izz="5e-04"/>
@@ -145,10 +143,8 @@
     <dynamics damping="0.7" friction="0.4"/>
     <limit effort="5000.0" lower="${-0.5*pi}" upper="${0.5*pi}" velocity="1"/>
-  </joint>
-  <link name="left_elbow">
+  </joint> -->
+  <!-- <link name="left_elbow">
     <inertial>
       <origin xyz="45.132e-3 -25.144e-3 -4.463e-3"/>
-      <!--mass value="0.096"/>
-      <inertia ixx="3.06e-05" ixy="2.52e-05" ixz="4.16e-07" iyy="1.39e-04" iyz="-4.01e-06" izz="1.46e-04"/-->
       <mass value="0.1"/>
       <inertia ixx="8.5833e-04" ixy="0" ixz="0" iyy="8.5833e-04" iyz="0" izz="5e-04"/>
@@ -172,10 +168,8 @@
     <dynamics damping="0.7" friction="0.4"/>
     <limit effort="5000.0" lower="${-pi}" upper="0" velocity="1"/>
-  </joint>
-  <link name="left_forearm">
+  </joint> -->
+  <!-- <link name="left_forearm">
     <inertial>
       <origin xyz="149.994e-3 -1.858e-3 0.041e-3"/>
-      <!--mass value="0.049"/>
-      <inertia ixx="6.72e-06" ixy="2.80e-06" ixz="-5.10e-08" iyy="9.24e-05" iyz="-1.64e-08" izz="9.39e-05"/-->
       <mass value="0.1"/>
       <inertia ixx="8.5833e-04" ixy="0" ixz="0" iyy="8.5833e-04" iyz="0" izz="5e-04"/>
@@ -199,10 +193,8 @@
     <dynamics damping="0.7" friction="0.4"/>
     <limit effort="5000.0" lower="${-0.5*pi}" upper="${0.5*pi}" velocity="1"/>
-  </joint>
-  <link name="left_wrist_pitch">
+  </joint> -->
+  <!-- <link name="left_wrist_pitch">
     <inertial>
       <origin xyz="0 0 0"/>
-      <!--mass value="0.049"/>
-      <inertia ixx="6.73e-06" ixy="-2.83e-06" ixz="-5.16e-08" iyy="9.42e-05" iyz="1.62e-08" izz="9.58e-05"/-->
       <mass value="0.021"/>
       <inertia ixx="8.5833e-04" ixy="0" ixz="0" iyy="8.5833e-04" iyz="0" izz="5e-04"/>
@@ -228,10 +220,8 @@
     <dynamics damping="0.7" friction="0.4"/>
     <limit effort="5000.0" lower="${-0.5*pi}" upper="${0.5*pi}" velocity="1"/>
-  </joint>
-  <link name="left_wrist_yaw">
+  </joint> -->
+  <!-- <link name="left_wrist_yaw">
     <inertial>
       <origin xyz="0 0 0"/>
-      <!--mass value="0.049"/>
-      <inertia ixx="6.73e-06" ixy="-2.83e-06" ixz="-5.16e-08" iyy="9.42e-05" iyz="1.62e-08" izz="9.58e-05"/-->
       <mass value="0.041"/>
       <inertia ixx="8.5833e-04" ixy="0" ixz="0" iyy="8.5833e-04" iyz="0" izz="5e-04"/>
@@ -257,174 +247,5 @@
     <dynamics damping="0.7" friction="0.4"/>
     <limit effort="5000.0" lower="${-0.5*pi}" upper="${0.5*pi}" velocity="1"/>
-  </joint>
-  <!-- Right arm -->
-  <!-- Inertias are not symmetrical, can't use xacro -->
-  <link name="right_shoulder">
-    <inertial>
-      <origin xyz="-14.08e-3 -0.409e-3 -28.745e-3"/>
-      <!--mass value="0.233"/>
-      <inertia ixx="6.70e-05" ixy="1.86e-06" ixz="-3.73e-06" iyy="8.45e-05" iyz="-1.19e-07" izz="9.90e-05"/-->
-      <mass value="0.1"/>
-      <inertia ixx="8.5833e-04" ixy="0" ixz="0" iyy="8.5833e-04" iyz="0" izz="5e-04"/>
-    </inertial>
-    <visual>
-      <geometry>
-        <mesh filename="package://robots_description/models/aeroarms/meshes/visual/right/shoulder.dae" scale=".001 .001 .001"/>
-      </geometry>
-    </visual>
-    <collision>
-      <geometry>
-        <mesh filename="package://robots_description/models/aeroarms/meshes/collision/right/shoulder.dae" scale=".001 .001 .001"/>
-      </geometry>
-    </collision>
-  </link>
-  <joint name="q2_1" type="revolute">
-    <!--origin xyz="200.781e-3 -124.765e-3 -123.775e-3"/-->
-    <origin xyz="50e-3 -120e-3 10e-3"/>
-    <parent link="base_link"/>
-    <child link="right_shoulder"/>
-    <axis xyz="0 0 1"/>
-    <dynamics damping="0.7" friction="0.4"/>
-    <limit effort="5000.0" lower="${-0.5*pi}" upper="${0.5*pi}" velocity="1"/>
-  </joint>
-  <link name="right_upperarm">
-    <inertial>
-      <origin xyz="-11.465e-3 -26.235e-3 -82.913e-3"/>
-      <!--mass value="0.244"/>
-      <inertia ixx="4.55e-04" ixy="2.46e-06" ixz="2.22e-05" iyy="4.76e-04" iyz="-2.48e-06" izz="9.24e-05"/-->
-      <mass value="0.1"/>
-      <inertia ixx="8.5833e-04" ixy="0" ixz="0" iyy="8.5833e-04" iyz="0" izz="5e-04"/>
-    </inertial>
-    <visual>
-      <geometry>
-        <mesh filename="package://robots_description/models/aeroarms/meshes/visual/right/upperarm.dae" scale=".001 .001 .001"/>
-      </geometry>
-    </visual>
-    <collision>
-      <geometry>
-        <mesh filename="package://robots_description/models/aeroarms/meshes/collision/right/upperarm.dae" scale=".001 .001 .001"/>
-      </geometry>
-    </collision>
-  </link>
-  <joint name="q2_2" type="revolute">
-    <origin xyz="0 -25.9e-3 -30e-3"/>
-    <parent link="right_shoulder"/>
-    <child link="right_upperarm"/>
-    <axis xyz="0 1 0"/>
-    <dynamics damping="0.7" friction="0.4"/>
-    <limit effort="5000.0" lower="${-0.5*pi}" upper="${0.5*pi}" velocity="1"/>
-  </joint>
-  <link name="right_elbow">
-    <inertial>
-      <origin xyz="45.132e-3 25.144e-3 -4.463e-3"/>
-      <!--mass value="0.096"/>
-      <inertia ixx="3.06e-05" ixy="-2.52e-05" ixz="4.16e-07" iyy="1.39e-04" iyz="4.01e-06" izz="1.46e-04"/-->
-      <mass value="0.1"/>
-      <inertia ixx="8.5833e-04" ixy="0" ixz="0" iyy="8.5833e-04" iyz="0" izz="5e-04"/>
-    </inertial>
-    <visual>
-      <geometry>
-        <mesh filename="package://robots_description/models/aeroarms/meshes/visual/right/elbow.dae" scale=".001 .001 .001"/>
-      </geometry>
-    </visual>
-    <collision>
-      <geometry>
-        <mesh filename="package://robots_description/models/aeroarms/meshes/collision/right/elbow.dae" scale=".001 .001 .001"/>
-      </geometry>
-    </collision>
-  </link>
-  <joint name="q2_3" type="revolute">
-    <origin xyz="0 -13e-3 -250e-3" rpy="0 ${0.5*pi} 0"/>
-    <parent link="right_upperarm"/>
-    <child link="right_elbow"/>
-    <axis xyz="0 1 0"/>
-    <dynamics damping="0.7" friction="0.4"/>
-    <limit effort="5000.0" lower="${-pi}" upper="0" velocity="1"/>
-  </joint>
-  <link name="right_forearm">
-    <inertial>
-      <origin xyz="149.597e-3 1.858e-3 0.041e-3"/>
-      <!--mass value="0.049"/>
-      <inertia ixx="6.73e-06" ixy="-2.83e-06" ixz="-5.16e-08" iyy="9.42e-05" iyz="1.62e-08" izz="9.58e-05"/-->
-      <mass value="0.1"/>
-      <inertia ixx="8.5833e-04" ixy="0" ixz="0" iyy="8.5833e-04" iyz="0" izz="5e-04"/>
-    </inertial>
-    <visual>
-      <geometry>
-        <mesh filename="package://robots_description/models/aeroarms/meshes/visual/right/forearm.dae" scale=".001 .001 .001"/>
-      </geometry>
-    </visual>
-    <collision>
-      <geometry>
-        <mesh filename="package://robots_description/models/aeroarms/meshes/collision/right/forearm.dae" scale=".001 .001 .001"/>
-      </geometry>
-    </collision>
-  </link>
-  <joint name="q2_4" type="revolute">
-    <origin xyz="80.9e-3 34.502e-3 0"/>
-    <parent link="right_elbow"/>
-    <child link="right_forearm"/>
-    <axis xyz="1 0 0"/>
-    <dynamics damping="0.7" friction="0.4"/>
-    <limit effort="5000.0" lower="${-0.5*pi}" upper="${0.5*pi}" velocity="1"/>
-  </joint>
-  <link name="right_wrist_pitch">
-    <inertial>
-      <origin xyz="0 0 0"/>
-      <!--mass value="0.049"/>
-      <inertia ixx="6.73e-06" ixy="-2.83e-06" ixz="-5.16e-08" iyy="9.42e-05" iyz="1.62e-08" izz="9.58e-05"/-->
-      <mass value="0.021"/>
-      <inertia ixx="8.5833e-04" ixy="0" ixz="0" iyy="8.5833e-04" iyz="0" izz="5e-04"/>
-    </inertial>
-    <visual>
-      <origin xyz="0 -32e-03 0"/>
-      <geometry>
-        <mesh filename="package://robots_description/models/aeroarms/meshes/visual/right/wrist_pitch.dae" scale=".001 .001 .001"/>
-      </geometry>
-    </visual>
-    <collision>
-      <origin xyz="0 -32e-03 0"/>
-      <geometry>
-        <mesh filename="package://robots_description/models/aeroarms/meshes/collision/right/wrist_pitch.dae" scale=".001 .001 .001"/>
-      </geometry>
-    </collision>
-  </link>
-  <joint name="q2_5" type="revolute">
-    <origin xyz="185e-03 2e-03 0" rpy="0 0 ${0.5*pi}"/>
-    <parent link="right_forearm"/>
-    <child link="right_wrist_pitch"/>
-    <axis xyz="1 0 0"/>
-    <dynamics damping="0.7" friction="0.4"/>
-    <limit effort="5000.0" lower="${-0.5*pi}" upper="${0.5*pi}" velocity="1"/>
-  </joint>
-  <link name="right_wrist_yaw">
-    <inertial>
-      <origin xyz="0 0 0"/>
-      <!--mass value="0.049"/>
-      <inertia ixx="6.73e-06" ixy="-2.83e-06" ixz="-5.16e-08" iyy="9.42e-05" iyz="1.62e-08" izz="9.58e-05"/-->
-      <mass value="0.041"/>
-      <inertia ixx="8.5833e-04" ixy="0" ixz="0" iyy="8.5833e-04" iyz="0" izz="5e-04"/>
-    </inertial>
-    <visual>
-      <origin xyz="0 -45e-03 0" rpy="0 0 ${0.5*pi}"/>
-      <geometry>
-        <mesh filename="package://robots_description/models/aeroarms/meshes/visual/right/wrist_yaw.dae" scale=".001 .001 .001"/>
-      </geometry>
-    </visual>
-    <collision>
-      <origin xyz="0 -45e-03 0" rpy="0 0 ${0.5*pi}"/>
-      <geometry>
-        <mesh filename="package://robots_description/models/aeroarms/meshes/collision/right/wrist_yaw.dae" scale=".001 .001 .001"/>
-      </geometry>
-    </collision>
-  </link>
-  <joint name="q2_6" type="revolute">
-    <origin xyz="0 0 0" rpy="0 0 0"/>
-    <parent link="right_wrist_pitch"/>
-    <child link="right_wrist_yaw"/>
-    <axis xyz="0 0 1"/>
-    <dynamics damping="0.7" friction="0.4"/>
-    <limit effort="5000.0" lower="${-0.5*pi}" upper="${0.5*pi}" velocity="1"/>
-  </joint>
+  </joint> -->
   <!-- Instantiate rotors -->
   <xacro:vertical_rotor

Commit message: Basic configuration for experiments. One arm centered, q1_2 pid tuned, urdf params modified. No collisions considered

File: robots_description/models/aeroarms/arm.transmission.xacro (robot description, xacro)
@@ -16,7 +16,7 @@
   <!-- Left arm -->
   <qside_x_transmission side="1" x="1"/>
-  <!-- <qside_x_transmission side="1" x="2"/> -->
-  <!-- <qside_x_transmission side="1" x="3"/>
-  <qside_x_transmission side="1" x="4"/> -->
+  <qside_x_transmission side="1" x="2"/>
+  <qside_x_transmission side="1" x="3"/>
+  <qside_x_transmission side="1" x="4"/>
   <!-- Right arm -->
   <!-- <qside_x_transmission side="2" x="1"/>

File: robots_description/models/aeroarms/geometry.xacro (robot description, xacro)
@@ -59,4 +59,5 @@
     <xacro:insert_block name="body_inertia" />
   </xacro:multirotor_base_macro>
+<!--
   <xacro:camera_macro
     namespace="${namespace}"
@@ -88,5 +89,5 @@
     <parent link="camera_depth_base_link"/>
     <child link="camera_depth_link"/>
-  </joint>
+  </joint> -->
   <!-- Left arm -->
   <!-- Inertias are not symmetrical, can't use xacro -->
@@ -104,20 +105,21 @@
       </geometry>
     </visual>
-    <collision>
+    <!-- <collision>
       <geometry>
         <mesh filename="package://robots_description/models/aeroarms/meshes/collision/left/shoulder.dae" scale=".001 .001 .001"/>
       </geometry>
-    </collision>
+    </collision> -->
   </link>
   <joint name="q1_1" type="revolute">
     <!--origin xyz="200.781e-3 125.235e-3 -123.775e-3"/-->
-    <origin xyz="50e-3 120e-3 10e-3"/>
+    <!-- <origin xyz="50e-3 120e-3 10e-3"/> -->
+    <origin xyz="0 0 -100e-3"/>
     <parent link="base_link"/>
     <child link="left_shoulder"/>
-    <axis xyz="0 1 0"/>
-    <dynamics damping="0.7" friction="0.4"/>
-    <limit effort="5000.0" lower="${-0.5*pi}" upper="${0.5*pi}" velocity="1"/>
-  </joint>
-  <!-- <link name="left_upperarm">
+    <axis xyz="1 0 0"/>
+    <dynamics damping="0.7" friction="0.4"/>
+    <limit effort="5.0" lower="${-0.5*pi}" upper="${0.5*pi}" velocity="1"/>
+  </joint>
+  <link name="left_upperarm">
     <inertial>
       <origin xyz="-10.426e-3 -26.142e-3 -82.655e-3"/>
@@ -130,9 +132,9 @@
       </geometry>
     </visual>
-    <collision>
+    <!-- <collision>
       <geometry>
         <mesh filename="package://robots_description/models/aeroarms/meshes/collision/left/upperarm.dae" scale=".001 .001 .001"/>
       </geometry>
-    </collision>
+    </collision> -->
   </link>
   <joint name="q1_2" type="revolute">
@@ -141,8 +143,8 @@
     <child link="left_upperarm"/>
     <axis xyz="0 1 0"/>
-    <dynamics damping="0.7" friction="0.4"/>
-    <limit effort="5000.0" lower="${-0.5*pi}" upper="${0.5*pi}" velocity="1"/>
-  </joint> -->
-  <!-- <link name="left_elbow">
+    <dynamics damping="0.0" friction="0.6"/>
+    <limit effort="5.5" lower="${-0.5*pi}" upper="${0.5*pi}" velocity="2.5"/>
+  </joint>
+  <link name="left_elbow">
     <inertial>
       <origin xyz="45.132e-3 -25.144e-3 -4.463e-3"/>
@@ -155,9 +157,9 @@
       </geometry>
     </visual>
-    <collision>
+    <!-- <collision>
       <geometry>
         <mesh filename="package://robots_description/models/aeroarms/meshes/collision/left/elbow.dae" scale=".001 .001 .001"/>
       </geometry>
-    </collision>
+    </collision> -->
   </link>
   <joint name="q1_3" type="revolute">
@@ -167,7 +169,7 @@
     <axis xyz="0 1 0"/>
     <dynamics damping="0.7" friction="0.4"/>
-    <limit effort="5000.0" lower="${-pi}" upper="0" velocity="1"/>
-  </joint> -->
-  <!-- <link name="left_forearm">
+    <limit effort="5.0" lower="${-pi}" upper="0" velocity="1"/>
+  </joint>
+  <link name="left_forearm">
     <inertial>
       <origin xyz="149.994e-3 -1.858e-3 0.041e-3"/>
@@ -180,9 +182,9 @@
       </geometry>
     </visual>
-    <collision>
+    <!-- <collision>
       <geometry>
         <mesh filename="package://robots_description/models/aeroarms/meshes/collision/left/forearm.dae" scale=".001 .001 .001"/>
       </geometry>
-    </collision>
+    </collision> -->
   </link>
   <joint name="q1_4" type="revolute">
@@ -192,11 +194,11 @@
     <axis xyz="1 0 0"/>
     <dynamics damping="0.7" friction="0.4"/>
-    <limit effort="5000.0" lower="${-0.5*pi}" upper="${0.5*pi}" velocity="1"/>
-  </joint> -->
-  <!-- <link name="left_wrist_pitch">
+    <limit effort="5.0" lower="${-0.5*pi}" upper="${0.5*pi}" velocity="1"/>
+  </joint>
+  <link name="left_wrist_pitch">
     <inertial>
       <origin xyz="0 0 0"/>
-      <mass value="0.021"/>
-      <inertia ixx="8.5833e-04" ixy="0" ixz="0" iyy="8.5833e-04" iyz="0" izz="5e-04"/>
+      <mass value="0.1"/>
+      <inertia ixx="8.5833e-04" ixy="0" ixz="0" iyy="8.5833e-04" iyz="0" izz="5.0e-04"/>
     </inertial>
     <visual>
@@ -206,10 +208,10 @@
       </geometry>
     </visual>
-    <collision>
+    <!-- <collision>
       <origin xyz="0 -32e-03 0"/>
       <geometry>
         <mesh filename="package://robots_description/models/aeroarms/meshes/collision/left/wrist_pitch.dae" scale=".001 .001 .001"/>
       </geometry>
-    </collision>
+    </collision> -->
   </link>
   <joint name="q1_5" type="revolute">
@@ -219,6 +221,6 @@
     <axis xyz="1 0 0"/>
     <dynamics damping="0.7" friction="0.4"/>
-    <limit effort="5000.0" lower="${-0.5*pi}" upper="${0.5*pi}" velocity="1"/>
-  </joint> -->
+    <limit effort="5.0" lower="${-0.5*pi}" upper="${0.5*pi}" velocity="1"/>
+  </joint>
   <!-- <link name="left_wrist_yaw">
     <inertial>
