Commit message: Change eef_mass from external call

File: robots_description/models/aeroarms/geometry.xacro (robot description, xacro)
@@ -199,5 +199,5 @@
     <inertial>
       <origin xyz="0 0 0"/>
-      <mass value="0.1"/>
+      <mass value="$(arg eef_mass)"/>
       <inertia ixx="8.5833e-04" ixy="0" ixz="0" iyy="8.5833e-04" iyz="0" izz="5.0e-04"/>
     </inertial>

File: robots_description/models/aeroarms/model.xacro (robot description, xacro)
@@ -13,4 +13,5 @@
   <xacro:arg name='enable_ground_truth' default='false' />
   <xacro:arg name='enable_logging' default='false' />
+  <xacro:arg name='eef_mass' default='0.1' />
   <!-- macros for gazebo plugins, sensors -->
   <xacro:include filename="$(find robots_description)/urdf/component_snippets.xacro" />
